File: pcb/CoolerMaster-USB-C.kicad_pcb (KiCad board)
At the start: 2 copper layers, 27.3 x 15 mm, 7 parts, among them J1 USB-C-SMD_C67381, J2 JST_SH_SM05B-SRSS-TB_1x05-1MP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, U1 USBLC6-2SC6

Commit message: Revision 1.3
Parts:
- added R2: , Keeb_components:R_0805, B.Cu at (129.6, 41.8)
- added REF**: breakaway-mousebites, Library:breakaway-mousebites, F.Cu at (117.7, 43.6)
Other:
- board size 27.3 x 15 mm -> 77.3 x 81.6 mm
- board text added: "Cooler Master 1.3"
- board text removed: "Cooler Master 1.2"
Changed lines of the file:
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@@
       (drillshape 0)
       (scaleselection 1)
-      (outputdirectory "./jlcpcbv1.2")
+      (outputdirectory "./jlcpcbv1.3")
     )
   )
@@
   (net 6 "Net-(J1-Pad5)")
   (net 7 "Net-(J1-Pad6)")
+  (footprint "Library:breakaway-mousebites" (layer "F.Cu")
+    (at 117.729 43.6 180)
+    (attr exclude_from_pos_files exclude_from_bom)
+    (fp_text reference "REF**" (at 0 -1.524) (layer "Dwgs.User")
+      (effects (font (size 1 1) (thickness 0.15)))
+    )
+    (fp_text value "breakaway-mousebites" (at 0 0.762) (layer "Dwgs.User")
+      (effects (font (size 1 1) (thickness 0.15)))
+    )
+    (fp_line (start 0 0) (end 2.54 -1.27) (layer "Cmts.User") (width 0.12))
+    (pad "" np_thru_hole circle (at 0 -0.254 180) (size 0.7874 0.7874) (drill 0.7874) (layers F&B.Cu *.Mask))
+    (pad "" np_thru_hole circle (at 2.54 -0.254 180) (size 0.7874 0.7874) (drill 0.7874) (layers F&B.Cu *.Mask))
+    (pad "" np_thru_hole circle (at 1.27 -0.254 180) (size 0.7874 0.7874) (drill 0.7874) (layers F&B.Cu *.Mask))
+    (pad "" np_thru_hole circle (at -1.27 -0.254 180) (size 0.7874 0.7874) (drill 0.7874) (layers F&B.Cu *.Mask))
+    (pad "" np_thru_hole circle (at -2.54 -0.254 180) (size 0.7874 0.7874) (drill 0.7874) (layers F&B.Cu *.Mask))
+  )
   (footprint "Keeb_components:R_0805" (layer "F.Cu")
     (at 125.349 41.148 -90)
@@
       ) (layer "B.Mask") (width 0) (fill solid))
   )
+  (footprint "Keeb_components:R_0805" (layer "B.Cu")
+    (at 129.583 41.783 180)
+    (descr "Resistor SMD 0805, reflow soldering, Vishay (see dcrcw.pdf)")
+    (tags "resistor 0805")
+    (property "Sheetfile" "980Daughterboard-USB-C.kicad_sch")
+    (property "Sheetname" "")
+    (attr smd)
+    (fp_text reference "R2" (at 0 1.5) (layer "B.Fab") hide
+      (effects (font (size 0.7 0.7) (thickness 0.15)) (justify mirror))
+    )
+    (fp_text value "" (at 0 1.651 unlocked) (layer "B.SilkS")
+      (effects (font (size 0.7 0.7) (thickness 0.15)) (justify mirror))
+    )
+    (fp_text user "${REFERENCE}" (at 0 0) (layer "B.Fab")
+      (effects (font (size 0.5 0.5) (thickness 0.075)) (justify mirror))
+    )
+    (fp_line (start 0.6 -0.88) (end -0.6 -0.88) (layer "B.SilkS") (width 0.12))
+    (fp_line (start -0.6 0.88) (end 0.6 0.88) (layer "B.SilkS") (width 0.12))
+    (fp_line (start 1.55 -0.9) (end -1.55 -0.9) (layer "B.CrtYd") (width 0.05))
+    (fp_line (start -1.55 0.9) (end -1.55 -0.9) (layer "B.CrtYd") (width 0.05))
+    (fp_line (start -1.55 0.9) (end 1.55 0.9) (layer "B.CrtYd") (width 0.05))
+    (fp_line (start 1.55 -0.9) (end 1.55 0.9) (layer "B.CrtYd") (width 0.05))
+    (fp_line (start 1 -0.62) (end -1 -0.62) (layer "B.Fab") (width 0.1))
+    (fp_line (start -1 -0.62) (end -1 0.62) (layer "B.Fab") (width 0.1))
+    (fp_line (start -1 0.62) (end 1 0.62) (layer "B.Fab") (width 0.1))
+    (fp_line (start 1 0.62) (end 1 -0.62) (layer "B.Fab") (width 0.1))
+    (pad "1" smd rect locked (at -1.1 0 180) (size 1.2 1.3) (layers "B.Cu" "B.Paste" "B.Mask")
+      (pintype "passive"))
+    (pad "2" smd rect locked (at 1.1 0 180) (size 1.2 1.3) (layers "B.Cu" "B.Paste" "B.Mask")
+      (pintype "passive"))
+    (model "${KIPRJMOD}/footprints.pretty/R0805.STEP"
+      (offset (xyz 0 0 0))
+      (scale (xyz 1 1 1))
+      (rotate (xyz 0 0 0))
+    )
+  )
   (gr_line (start 112.48 29.1376) (end 112.48 30.9376) (layer "Edge.Cuts") (width 0.15))
   (gr_arc (start 111.98 28.6376) (mid 112.349497 28.768102) (end 112.48 29.1376) (layer "Edge.Cuts") (width 0.15))
@@
   (gr_arc (start 126.2888 34.1376) (mid 125.935247 33.991153) (end 125.7888 33.6376) (layer "Edge.Cuts") (width 0.15))
   (gr_line (start 111.98 28.6376) (end 105.2888 28.6376) (layer "Edge.Cuts") (width 0.15))
+  (gr_line (start 157.08 22) (end 132.969 22) (layer "Edge.Cuts") (width 0.15))
   (gr_circle (center 109.98 31.4376) (end 108.38 31.3376) (layer "Edge.Cuts") (width 0.15) (fill none))
   (gr_arc (start 112.98 31.4376) (mid 112.640958 31.276642) (end 112.48 30.9376) (layer "Edge.Cuts") (width 0.15))
+  (gr_line (start 79.7888 22) (end 79.7888 103.6376) (layer "Edge.Cuts") (width 0.15))
   (gr_circle (center 128.83 37.3876) (end 130.43 37.3876) (layer "Edge.Cuts") (width 0.15) (fill none))
+  (gr_line (start 132.969 44.1376) (end 132.969 22) (layer "Edge.Cuts") (width 0.15))
   (gr_arc (start 104.7888 29.1376) (mid 104.935247 28.784047) (end 105.2888 28.6376) (layer "Edge.Cuts") (width 0.15))
   (gr_line (start 123.94 31.4376) (end 125.2888 31.4376) (layer "Edge.Cuts") (width 0.15))
+  (gr_line (start 120.904 44.1376) (end 120.904 43.6) (layer "Edge.Cuts") (width 0.15))
   (gr_line (start 132.08 34.6376) (end 132.08 43.1376) (layer "Edge.Cuts") (width 0.15))
   (gr_line (start 112.98 31.4376) (end 114.01 31.4376) (layer "Edge.Cuts") (width 0.15))
-  (gr_line (start 131.58 43.6376) (end 112.48 43.6376) (layer "Edge.Cuts") (width 0.15))
+  (gr_line (start 103.7888 22) (end 103.7888 44.1376) (layer "Edge.Cuts") (width 0.15))
+  (gr_line (start 79.7888 22) (end 103.7888 22) (layer "Edge.Cuts") (width 0.15))
+  (gr_line (start 120.904 44.1376) (end 132.969 44.1376) (layer "Edge.Cuts") (width 0.15))
+  (gr_line (start 131.58 43.6376) (end 120.904 43.6) (layer "Edge.Cuts") (width 0.15))
   (gr_arc (start 105.2888 43.6376) (mid 104.935247 43.491153) (end 104.7888 43.1376) (layer "Edge.Cuts") (width 0.15))
-  (gr_line (start 105.2888 43.6376) (end 112.48 43.6376) (layer "Edge.Cuts") (width 0.15))
+  (gr_line (start 105.2888 43.6376) (end 114.3 43.561) (layer "Edge.Cuts") (width 0.15))
+  (gr_line (start 79.7888 103.6376) (end 157.08 103.6376) (layer "Edge.Cuts") (width 0.15))
   (gr_arc (start 114.01 31.4376) (mid 114.363553 31.584047) (end 114.51 31.9376) (layer "Edge.Cuts") (width 0.15))
   (gr_arc (start 132.08 43.1376) (mid 131.933553 43.491153) (end 131.58 43.6376) (layer "Edge.Cuts") (width 0.15))
+  (gr_line (start 120.904 43.688) (end 120.904 43.688) (layer "Edge.Cuts") (width 0.15))
   (gr_line (start 123.44 31.9376) (end 123.44 32.0776) (layer "Edge.Cuts") (width 0.15))
   (gr_line (start 126.2888 34.1376) (end 131.58 34.1376) (layer "Edge.Cuts") (width 0.15))
+  (gr_line (start 114.3 44.1376) (end 103.7888 44.1376) (layer "Edge.Cuts") (width 0.15))
+  (gr_line (start 157.08 22) (end 157.08 103.6376) (layer "Edge.Cuts") (width 0.15))
+  (gr_line (start 114.3 43.561) (end 114.3 44.1376) (layer "Edge.Cuts") (width 0.15))
   (gr_line (start 104.7888 29.1376) (end 104.7888 43.1376) (layer "Edge.Cuts") (width 0.15))
   (gr_arc (start 123.44 31.9376) (mid 123.586447 31.584047) (end 123.94 31.4376) (layer "Edge.Cuts") (width 0.15))
   (gr_arc (start 131.58 34.1376) (mid 131.933553 34.284047) (end 132.08 34.6376) (layer "Edge.Cuts") (width 0.15))
   (gr_arc (start 125.2888 31.4376) (mid 125.633357 31.593043) (end 125.7888 31.9376) (layer "Edge.Cuts") (width 0.15))
-  (gr_text "Cooler Master 1.2" (at 118.98 41.91) (layer "B.SilkS")
+  (gr_text "Cooler Master 1.3" (at 118.98 41.91) (layer "B.SilkS")
     (effects (font (size 1 1) (thickness 0.15)) (justify mirror))
   )
@@
     (polygon
       (pts
-        (xy 146.538 46.1318)
-        (xy 101.453 46.1318)
-        (xy 101.453 -1.671)
-        (xy 146.538 -1.798)
+        (xy 133.477 43.942)
+        (xy 103.505 43.942)
+        (xy 103.505 27.686)
+        (xy 133.477 27.686)
       )
     )
@@
     (polygon
       (pts
-        (xy 145.950306 46.335286)
-        (xy 101.627306 46.208286)
-        (xy 101.707 -1.417)
-        (xy 146.238188 -1.290944)
+        (xy 133.477 43.942)
+        (xy 103.505 43.942)
+        (xy 103.505 27.686)
+        (xy 133.477 27.686)
       )
     )

Commit message: Version 1.4
Version 1.4
Parts:
- removed REF**: breakaway-mousebites, Library:breakaway-mousebites
Other:
- board size 77.3 x 81.6 mm -> 27.3 x 15 mm
- board text added: "Cooler Master 1.4"
- board text removed: "Cooler Master 1.3"
Changed lines of the file:
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@@
   (net 6 "Net-(J1-Pad5)")
   (net 7 "Net-(J1-Pad6)")
-  (footprint "Library:breakaway-mousebites" (layer "F.Cu")
-    (at 117.729 43.6 180)
-    (attr exclude_from_pos_files exclude_from_bom)
-    (fp_text reference "REF**" (at 0 -1.524) (layer "Dwgs.User")
-      (effects (font (size 1 1) (thickness 0.15)))
-    )
-    (fp_text value "breakaway-mousebites" (at 0 0.762) (layer "Dwgs.User")
-      (effects (font (size 1 1) (thickness 0.15)))
-    )
-    (fp_line (start 0 0) (end 2.54 -1.27) (layer "Cmts.User") (width 0.12))
-    (pad "" np_thru_hole circle (at 0 -0.254 180) (size 0.7874 0.7874) (drill 0.7874) (layers F&B.Cu *.Mask))
-    (pad "" np_thru_hole circle (at 2.54 -0.254 180) (size 0.7874 0.7874) (drill 0.7874) (layers F&B.Cu *.Mask))
-    (pad "" np_thru_hole circle (at 1.27 -0.254 180) (size 0.7874 0.7874) (drill 0.7874) (layers F&B.Cu *.Mask))
-    (pad "" np_thru_hole circle (at -1.27 -0.254 180) (size 0.7874 0.7874) (drill 0.7874) (layers F&B.Cu *.Mask))
-    (pad "" np_thru_hole circle (at -2.54 -0.254 180) (size 0.7874 0.7874) (drill 0.7874) (layers F&B.Cu *.Mask))
-  )
   (footprint "Keeb_components:R_0805" (layer "F.Cu")
     (at 125.349 41.148 -90)
@@
   (gr_arc (start 126.2888 34.1376) (mid 125.935247 33.991153) (end 125.7888 33.6376) (layer "Edge.Cuts") (width 0.15))
   (gr_line (start 111.98 28.6376) (end 105.2888 28.6376) (layer "Edge.Cuts") (width 0.15))
-  (gr_line (start 157.08 22) (end 132.969 22) (layer "Edge.Cuts") (width 0.15))
   (gr_circle (center 109.98 31.4376) (end 108.38 31.3376) (layer "Edge.Cuts") (width 0.15) (fill none))
   (gr_arc (start 112.98 31.4376) (mid 112.640958 31.276642) (end 112.48 30.9376) (layer "Edge.Cuts") (width 0.15))
-  (gr_line (start 79.7888 22) (end 79.7888 103.6376) (layer "Edge.Cuts") (width 0.15))
   (gr_circle (center 128.83 37.3876) (end 130.43 37.3876) (layer "Edge.Cuts") (width 0.15) (fill none))
-  (gr_line (start 132.969 44.1376) (end 132.969 22) (layer "Edge.Cuts") (width 0.15))
   (gr_arc (start 104.7888 29.1376) (mid 104.935247 28.784047) (end 105.2888 28.6376) (layer "Edge.Cuts") (width 0.15))
   (gr_line (start 123.94 31.4376) (end 125.2888 31.4376) (layer "Edge.Cuts") (width 0.15))
-  (gr_line (start 120.904 44.1376) (end 120.904 43.6) (layer "Edge.Cuts") (width 0.15))
   (gr_line (start 132.08 34.6376) (end 132.08 43.1376) (layer "Edge.Cuts") (width 0.15))
   (gr_line (start 112.98 31.4376) (end 114.01 31.4376) (layer "Edge.Cuts") (width 0.15))
-  (gr_line (start 103.7888 22) (end 103.7888 44.1376) (layer "Edge.Cuts") (width 0.15))
-  (gr_line (start 79.7888 22) (end 103.7888 22) (layer "Edge.Cuts") (width 0.15))
-  (gr_line (start 120.904 44.1376) (end 132.969 44.1376) (layer "Edge.Cuts") (width 0.15))
   (gr_line (start 131.58 43.6376) (end 120.904 43.6) (layer "Edge.Cuts") (width 0.15))
   (gr_arc (start 105.2888 43.6376) (mid 104.935247 43.491153) (end 104.7888 43.1376) (layer "Edge.Cuts") (width 0.15))
-  (gr_line (start 105.2888 43.6376) (end 114.3 43.561) (layer "Edge.Cuts") (width 0.15))
-  (gr_line (start 79.7888 103.6376) (end 157.08 103.6376) (layer "Edge.Cuts") (width 0.15))
+  (gr_line (start 105.2888 43.6376) (end 120.904 43.6) (layer "Edge.Cuts") (width 0.15))
   (gr_arc (start 114.01 31.4376) (mid 114.363553 31.584047) (end 114.51 31.9376) (layer "Edge.Cuts") (width 0.15))
   (gr_arc (start 132.08 43.1376) (mid 131.933553 43.491153) (end 131.58 43.6376) (layer "Edge.Cuts") (width 0.15))
-  (gr_line (start 120.904 43.688) (end 120.904 43.688) (layer "Edge.Cuts") (width 0.15))
   (gr_line (start 123.44 31.9376) (end 123.44 32.0776) (layer "Edge.Cuts") (width 0.15))
   (gr_line (start 126.2888 34.1376) (end 131.58 34.1376) (layer "Edge.Cuts") (width 0.15))
-  (gr_line (start 114.3 44.1376) (end 103.7888 44.1376) (layer "Edge.Cuts") (width 0.15))
-  (gr_line (start 157.08 22) (end 157.08 103.6376) (layer "Edge.Cuts") (width 0.15))
-  (gr_line (start 114.3 43.561) (end 114.3 44.1376) (layer "Edge.Cuts") (width 0.15))
   (gr_line (start 104.7888 29.1376) (end 104.7888 43.1376) (layer "Edge.Cuts") (width 0.15))
   (gr_arc (start 123.44 31.9376) (mid 123.586447 31.584047) (end 123.94 31.4376) (layer "Edge.Cuts") (width 0.15))
   (gr_arc (start 131.58 34.1376) (mid 131.933553 34.284047) (end 132.08 34.6376) (layer "Edge.Cuts") (width 0.15))
   (gr_arc (start 125.2888 31.4376) (mid 125.633357 31.593043) (end 125.7888 31.9376) (layer "Edge.Cuts") (width 0.15))
-  (gr_text "Cooler Master 1.3" (at 118.98 41.91) (layer "B.SilkS")
+  (gr_text "Cooler Master 1.4" (at 118.98 41.91) (layer "B.SilkS")
     (effects (font (size 1 1) (thickness 0.15)) (justify mirror))
   )
